Commit message: Coffee Table position fixed

File: src/baxter_chess_game/models/cafe_table.xacro (robot description, xacro)
@@ -4,9 +4,9 @@
     <inertial>
       <mass value="0"/>
-      <origin rpy="0  0  0" xyz="0  0  0"/>
+      <origin rpy="0  0  0" xyz="-0.25  0.45  0"/>
       <inertia ixx="0" ixy="0" ixz="0" iyy="0" iyz="0" izz="0"/>
     </inertial>
     <collision name="cafe_table__surface">
-      <origin rpy="0  0  0" xyz="0     0     0.755"/>
+      <origin rpy="0  0  0" xyz="-0.25     0.45     0.755"/>
       <geometry>
         <box size="0.913 0.913 0.04"/>
@@ -14,5 +14,5 @@
     </collision>
     <collision name="cafe_table__column">
-      <origin rpy="0  0  0" xyz="0    0    0.37"/>
+      <origin rpy="0  0  0" xyz="-0.25    0.45    0.37"/>
       <geometry>
         <box size="0.042 0.042 0.74"/>
@@ -20,5 +20,5 @@
     </collision>
     <collision name="cafe_table__base">
-      <origin rpy="0  0  0" xyz="0    0    0.02"/>
+      <origin rpy="0  0  0" xyz="-0.25    0.45    0.02"/>
       <geometry>
         <box size="0.56 0.56 0.04"/>
@@ -26,5 +26,5 @@
     </collision>
     <visual name="cafe_table__visual">
-      <origin rpy="0  0  0" xyz="0  0  0"/>
+      <origin rpy="0  0  0" xyz="-0.25  0.45  0"/>
       <geometry>
         <mesh filename="package://baxter_sim_examples/models/cafe_table/meshes/cafe_table.dae" scale="1.0 1.0 1.0"/>

Commit message: Completed

File: src/baxter_chess_game/models/cafe_table.xacro (robot description, xacro)
@@ -4,9 +4,9 @@
     <inertial>
       <mass value="0"/>
-      <origin rpy="0  0  0" xyz="-0.25  0.45  0"/>
+      <origin rpy="0  0  0" xyz="-0.26  0.45  0"/>
       <inertia ixx="0" ixy="0" ixz="0" iyy="0" iyz="0" izz="0"/>
     </inertial>
     <collision name="cafe_table__surface">
-      <origin rpy="0  0  0" xyz="-0.25     0.45     0.755"/>
+      <origin rpy="0  0  0" xyz="-0.26     0.45     0.755"/>
       <geometry>
         <box size="0.913 0.913 0.04"/>
@@ -14,5 +14,5 @@
     </collision>
     <collision name="cafe_table__column">
-      <origin rpy="0  0  0" xyz="-0.25    0.45    0.37"/>
+      <origin rpy="0  0  0" xyz="-0.26    0.45    0.37"/>
       <geometry>
         <box size="0.042 0.042 0.74"/>
@@ -20,5 +20,5 @@
     </collision>
     <collision name="cafe_table__base">
-      <origin rpy="0  0  0" xyz="-0.25    0.45    0.02"/>
+      <origin rpy="0  0  0" xyz="-0.26    0.45    0.02"/>
       <geometry>
         <box size="0.56 0.56 0.04"/>
@@ -26,5 +26,5 @@
     </collision>
     <visual name="cafe_table__visual">
-      <origin rpy="0  0  0" xyz="-0.25  0.45  0"/>
+      <origin rpy="0  0  0" xyz="-0.26  0.45  0"/>
       <geometry>
         <mesh filename="package://baxter_sim_examples/models/cafe_table/meshes/cafe_table.dae" scale="1.0 1.0 1.0"/>
